File: Hardware/Heep_TPLinkBackpack_Proto/Teensy_backpack_proto.brd (EAGLE design)
At the start: 45 x 57.5 mm, 30 parts, among them Q1 25MHz, Q2 600mA/40V, U1 ENC28J60-SO

Commit message: #44 almost done with board design
Parts:
- removed Q1: 25MHz, adafruit:SM49
- added BREAKOUT1, BREAKOUT2: (no value), SparkFun-Connectors:1X14
- added C8: 10uF, SparkFun-Passives:0603-CAP
- added JP10, JP8, JP9: (no value), SparkFun-Connectors:2X5_NOSILK
- added Q3: (no value), adafruit:NX3225
- added R8: 100, SparkFun-Resistors:0603-RES
- D1, D2, D3: device SparkFun-DiscreteSemi:DIODE-1N4148 -> adafruit:SOD-123
- JP3: device SparkFun-Connectors:1X04_NO_SILK_ALL_ROUND -> SparkFun-Connectors:2X5_NOSILK
- JP5: device SparkFun-Connectors:1X03 -> SparkFun-Connectors:2X5_NOSILK
- JP6, JP7: device SparkFun-Connectors:1X01 -> SparkFun-Connectors:2X5_NOSILK
- Q2: device SparkFun-DiscreteSemi:TO-92 -> microbuilder:SOT23-R
- U1: value ENC28J60-SO -> ENC28J60-SSOP; device microchip-enc28j60:SO28W -> microchip-enc28j60:SSOP28
- moved JP3 60.7 mm to (3.84, 50.5), turned to 0 degrees
- moved JP6 41.5 mm to (3.84, 37.8)
- moved C3 33.4 mm to (33.9, 3.88), turned to 270 degrees
- moved C4 31.2 mm to (39.5, 3.91), turned to 270 degrees
- moved JP5 28.6 mm to (8.92, 50.5)
- moved C6 27.6 mm to (42.8, 6.69)
- moved R5 26.9 mm to (17.4, 25.7), turned to 270 degrees
- moved C7 26.8 mm to (42.8, 4.94)
- moved Q2 26.3 mm to (31.1, 52.1), turned to 90 degrees
- moved C5 26.2 mm to (42.8, 3.14)
- moved R4 20.9 mm to (29.3, 18.9), turned to 180 degrees
- moved D1 20.8 mm to (31.0, 46.3), turned to 180 degrees
- moved C2 16.9 mm to (28.3, 5.67), turned to 90 degrees
- moved C10 15.9 mm to (43.0, 19.1), turned to 180 degrees
- moved D2 15.6 mm to (31.0, 48.5), turned to 0 degrees
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Connections:
- removed net VIN: U$1.VIN
- new net N$10: BREAKOUT2.7, U$1.6
- new net N$11: BREAKOUT2.8, U$1.5
- new net N$14: BREAKOUT2.9, U$1.4
- new net N$16: BREAKOUT2.10, U$1.3
- new net N$18: BREAKOUT2.12, U$1.1
- new net N$19: BREAKOUT2.13, U$1.0
- new net N$20: BREAKOUT1.4, U$1.23/A9
- new net N$21: BREAKOUT1.5, U$1.22/A8
- new net N$22: BREAKOUT1.6, U$1.21/A7
- new net N$23: BREAKOUT1.7, U$1.20/A6
- new net N$24: BREAKOUT1.8, U$1.19/A5
- new net N$25: BREAKOUT1.9, U$1.18/A4
- new net N$26: BREAKOUT1.10, U$1.17/A3
- new net N$27: BREAKOUT1.11, U$1.16/A2
- new net N$28: BREAKOUT1.12, U$1.15/A1
- new net N$29: BREAKOUT1.13, U$1.14/A0
- new net N$4: D3.A, R8.1
- new net N$6: BREAKOUT2.4, U$1.9
- new net N$8: BREAKOUT2.5, U$1.8
- new net N$9: BREAKOUT2.6, U$1.7
- new net TEENSY_VIN: BREAKOUT1.1, U$1.VIN
- net #CS: now also BREAKOUT2.3; no longer JP5.1
- net #RESET: now also BREAKOUT2.11; no longer JP7.1
- net 3.3V: now also BREAKOUT1.3, C8.1, JP10.1, JP10.3, JP10.5, JP10.7, JP10.9, R8.2; no longer D3.A
- net AGND: now also BREAKOUT1.2, C1.2, C10.1, C2.2, C3.2, C4.2, C5.2, C6.2, C7.2, C8.2, JP10.10, JP10.2, JP10.4, JP10.6, JP10.8, Q2.2, Q3.2, Q3.4, R7.2, U1.11, U1.18, U1.2, U1.21, U1.22; no longer Q2.3
- net GND: now also BREAKOUT2.14, Q2.3; no longer C1.2, C10.1, C2.2, C3.2, C4.2, C5.2, C6.2, C7.2, Q2.1, R7.2, U1.11, U1.18, U1.2, U1.21, U1.22
- net N$1: now also D1.C, D2.A; no longer D1.A, D2.C
- net N$12: now also Q3.1; no longer Q1.2
- net N$13: now also Q3.3; no longer Q1.1
- net N$2: now also D2.C, Q2.1; no longer D1.C, Q2.2
- net N$3: now also D1.A; no longer D2.A
- net RD+: no longer JP3.3
- net RD-: no longer JP3.4
- net SCK: now also BREAKOUT1.14; no longer JP6.1
- net SI: now also BREAKOUT2.2; no longer JP5.2
- net SO: now also BREAKOUT2.1; no longer JP5.3
- net TD+: no longer JP3.2
- net TD-: no longer JP3.1
Routing:
- net AGND: track 26.6 -> 145.7 mm, vias 0 -> 6
- net GND: track 121.9 -> 11.1 mm
- net 3.3V: track 138.1 -> 167.0 mm, vias 0 -> 4
- net RD-: track 36.9 -> 11.0 mm
- net N$12: track 32.1 -> 8.69 mm
- net #RESET: track 22.0 -> 43.5 mm, vias 0 -> 2
- net SI: track 4.13 -> 22.2 mm, vias 0 -> 2
- net SO: track 4.13 -> 22.0 mm
- net N$13: track 25.9 -> 10.7 mm
- net N$15: track 2.60 -> 15.5 mm, vias 0 -> 2
- net TD-: track 21.9 -> 34.5 mm, vias 0 -> 2
- net RD+: track 24.9 -> 14.8 mm, vias 0 -> 2
- net #CS: track 15.8 -> 25.4 mm, vias 0 -> 1
- net SCK: track 4.61 -> 12.8 mm, vias 0 -> 1
- net N$5: track 25.9 -> 19.8 mm, vias 0 -> 2
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
Commit message: #44 ready for dylan check
Parts:
- moved C3 0.60 mm to (33.9, 4.48)
- moved C4 0.60 mm to (39.5, 4.51)
- moved Q3 0.60 mm to (36.8, 3.30)
- moved R5 0.51 mm to (17.9, 25.8)
- moved C7 0.36 mm to (43.0, 5.24)
- moved C8 0.36 mm to (43.0, 1.70)
- moved C6 0.36 mm to (43.0, 6.99)
- moved C5 0.36 mm to (43.0, 3.44)
Routing:
- net AGND: track 145.7 -> 168.6 mm, vias 6 -> 5
- net N$5: track 19.8 -> 21.5 mm
- net 3.3V: track 167.0 -> 167.7 mm
- net N$13: track 10.7 -> 10.1 mm
- net #CS: track 25.4 -> 24.8 mm
- added copper zone on layer 1, net AGND
Other:
- outline, holes or cut-outs redrawn
- board text added: "HEEP.IO"
