File: Hardware/Heep_TPLinkBackpack_Relay/Teensy_backpack_relay.brd (EAGLE design)
At the start: 45 x 87 mm, 49 parts, among them K1 G5LE, K2 G5LE, Q1 MMBT2222, Q2 600mA/40V, Q4 MMBT2222, U1 ENC28J60-SSOP

Commit message: #260 Change teensy capacitors to 8pf
Parts:
- C3, C4: value 10pF -> 8pF
Changed lines of the file:
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@@
 <attribute name="VALUE" x="30.3509" y="20.088228125" size="1.016" layer="27" font="vector" rot="R180"/>
 </element>
-<element name="C3" library="SparkFun-Passives" package="0603-CAP" value="10pF" x="33.927371875" y="4.4812625" smashed="yes" rot="R270">
+<element name="C3" library="SparkFun-Passives" package="0603-CAP" value="8pF" x="33.927371875" y="4.4812625" smashed="yes" rot="R270">
 <attribute name="NAME" x="34.689371875" y="5.3702625" size="0.4064" layer="25" font="vector" rot="R270"/>
 <attribute name="VALUE" x="33.384371875" y="6.7972625" size="1.016" layer="27" font="vector" rot="R270"/>
 </element>
-<element name="C4" library="SparkFun-Passives" package="0603-CAP" value="10pF" x="39.4513125" y="4.50935625" smashed="yes" rot="R270">
+<element name="C4" library="SparkFun-Passives" package="0603-CAP" value="8pF" x="39.4513125" y="4.50935625" smashed="yes" rot="R270">
 <attribute name="NAME" x="40.2133125" y="5.39835625" size="0.4064" layer="25" font="vector" rot="R270"/>
 <attribute name="VALUE" x="39.1083125" y="5.92535625" size="1.016" layer="27" font="vector" rot="R270"/>
