File: Hardware/PIC18f26k40_TPLinkBackpack/PIC18f26k40_TPLinkBackpack.brd (EAGLE design)
At the start: 45 x 57.5 mm, 46 parts, among them IC1 PIC18F2480-I/ML, U1 W5500

Commit message: HEEP-299 WIP
Parts:
- removed J3, J4: (no value), SparkFun-Connectors:1X14
- added C21, C25: (no value), SparkFun-Capacitors:0603-CAP
- added J2, J8: (no value), SparkFun-Connectors:SCREWTERMINAL-5MM-2
- added J6, J7: (no value), SparkFun-Connectors:1X02
- added JP1, JP2, JP4, JP7: (no value), SparkFun-Connectors:1X03_LONGPADS
- added OK1, OK2: MOC3042T, optocoupler:DIL06B
- added R12, R13, R14, R15, R25, R26, R27, R28: 100k, SparkFun-Resistors:0603
- added T1, T2: BT138-V, triac:TO220BV
- J5: device SparkFun-Connectors:1X02 -> SparkFun-Connectors:1X02@1
- JP3: device SparkFun-Connectors:1X02_NO_SILK -> SparkFun-Connectors:1X02_NO_SILK@1
- moved LED1 80.8 mm to (72.0, 27.1)
- moved R7 80.5 mm to (77.8, 24.7)
- moved LED2 80.3 mm to (65.4, 27.2)
- moved R6 74.3 mm to (73.4, 21.4)
- moved IC1 59.7 mm to (8.71, 14.2), turned to 0 degrees
- moved J5 31.2 mm to (63.6, 21.9)
- moved U1 21.1 mm to (37.4, 14.4), turned to 270 degrees
- moved C13 17.7 mm to (76.0, 15.5)
- moved C10 17.7 mm to (56.9, 15.5)
- moved C11 17.7 mm to (63.3, 15.5)
- moved C12 17.7 mm to (69.6, 15.5)
- moved C14 17.7 mm to (82.3, 15.5)
- moved C15 17.7 mm to (88.7, 15.5)
- moved C16 17.7 mm to (95.0, 15.5)
- moved C17 17.7 mm to (101.4, 15.5)
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Connections:
- new net CAPTORES1: C25.1, R27.1
- new net CAPTORES2: C21.1, R14.1
- new net GATE1: OK1.4, R26.2, T1.G
- new net GATE2: OK2.4, R13.2, T2.G
- new net LIVE: AC_L.P$1, R12.2, R14.2, R25.2, R27.2, T1.T2, T2.T2
- new net LOAD1: C25.2, J8.2, R26.1, T1.T1
- new net LOAD2: C21.2, J2.2, R13.1, T2.T1
- new net N$10: OK2.1, R15.1
- new net N$12: J6.1, OK2.2
- new net N$18: OK1.1, R28.1
- new net N$19: J7.1, OK1.2
- new net N$3: J7.2, R28.2
- new net N$8: J6.2, R15.2
- new net NEUTRAL: AC_N.P$1, J2.1, J8.1
- new net RESTOMOC1: OK1.6, R25.1
- new net RESTOMOC2: OK2.6, R12.1
- net GND: no longer J3.7, J4.5
- net MCLR: no longer J3.14
- net MISO: no longer J4.1
- net MOSI: no longer J4.2
- net PGC: no longer J4.13
- net PGD: no longer J4.14
- net RA0: no longer J3.13
- net RA1: no longer J3.12
- net RA2: no longer J3.11
- net RA3: no longer J3.10
- net RA4: no longer J3.9
- net RA5: no longer J3.8
- net RA6: no longer J3.5
- net RA7: no longer J3.6
- net RB0: no longer J4.7
- net RB1: no longer J4.8
- net RB2: no longer J4.9
- net RB3: no longer J4.10
- net RB4: no longer J4.11
- net RB5: no longer J4.12
- net RC1: no longer J3.3
- net RC2: no longer J3.2
- net RC6: no longer J4.3
- net RC7: no longer J4.4
- net SCK: no longer J3.1
- net SCSN: no longer J3.4
- net VCC: no longer J4.6
Routing:
- net RESTOMOC2: track 0.00 -> 3.30 mm
