File: Hardware/PIC18f26k40_TPLinkBackpack/PIC18f26k40_TPLinkBackpack.sch (EAGLE design)
At the start: 46 parts, among them IC1 PIC18F2480-I/ML, U1 W5500

Commit message: HEEP-299 WIP
Parts:
- removed J3, J4: (no value), SparkFun-Connectors:CONN_14
- added C21, C25: (no value), SparkFun-Capacitors:CAP0603-CAP
- added J2, J8: (no value), SparkFun-Connectors:CONN_025MM
- added J6, J7: (no value), SparkFun-Connectors:CONN_02
- added JP1, JP2, JP4, JP7: (no value), SparkFun-Connectors:M03LONGPADS
- added OK1, OK2: MOC3042T, optocoupler:MOC3042T
- added R12, R13, R14, R15, R25, R26, R27, R28: 100k, SparkFun-Resistors:100KOHM-0603-1/10W-1%
- added T1, T2: BT138-V, triac:BT138-V
Connections:
- new net CAPTORES1: C25.1, R27.1
- new net CAPTORES2: C21.1, R14.1
- new net GATE1: OK1.A1, R26.2, T1.G
- new net GATE2: OK2.A1, R13.2, T2.G
- new net LIVE: AC_L.AC, R12.2, R14.2, R25.2, R27.2, T1.A2, T2.A2
- new net LOAD1: C25.2, J8.2, R26.1, T1.A1
- new net LOAD2: C21.2, J2.2, R13.1, T2.A1
- new net N$10: OK2.A, R15.1
- new net N$12: J6.1, OK2.C
- new net N$18: OK1.A, R28.1
- new net N$19: J7.1, OK1.C
- new net N$3: J7.2, R28.2
- new net N$8: J6.2, R15.2
- new net NEUTRAL: AC_N.AC, J2.1, J8.1
- new net RESTOMOC1: OK1.A2, R25.1
- new net RESTOMOC2: OK2.A2, R12.1
- net GND: no longer J3.7, J4.5
- net MCLR: no longer J3.14
- net MISO: no longer J4.1
- net MOSI: no longer J4.2
- net PGC: no longer J4.13
- net PGD: no longer J4.14
- net RA0: no longer J3.13
- net RA1: no longer J3.12
- net RA2: no longer J3.11
- net RA3: no longer J3.10
- net RA4: no longer J3.9
- net RA5: no longer J3.8
- net RA6: no longer J3.5
- net RA7: no longer J3.6
- net RB0: no longer J4.7
- net RB1: no longer J4.8
- net RB2: no longer J4.9
- net RB3: no longer J4.10
- net RB4: no longer J4.11
- net RB5: no longer J4.12
- net RC1: no longer J3.3
- net RC2: no longer J3.2
- net RC6: no longer J4.3
- net RC7: no longer J4.4
- net SCK: no longer J3.1
- net SCSN: no longer J3.4
- net VCC: no longer J4.6
