File: Hardware/PIC18f26k40_TPBackpack/REV B/PIC_backpack.brd (EAGLE design)
At the start: 45 x 57.5 mm, 61 parts, among them IC1 PIC18F2480-I/ML, T1 BT138-V, T2 BT138-V, U4 W5500, Y2 CRYSTAL-GROUNDEDSMD-3.2X2.5

Commit message: HEEP-414 back to work
Parts:
- removed T2: BT138-V, triac:TO220BV
- added T3: BT138, triac:D2PAK-3
- added U1: 4MB Flash, SparkFun-IC-Memory:SO08
- T1: value BT138-V -> BT138; device triac:TO220BV -> triac:D2PAK-3
- U$1: value TPLINK_BACKPACK -> TPLINK_BACKPACKMINIMAL_HOLES; device Heep:BACKPACK_WITH_PROTO -> Heep:BACKPACK_MINIMAL_HOLES
- moved T1 15.7 mm to (11.1, 51.3)
- moved U$14 10.6 mm to (10.2, 5.08), turned to 180 degrees
- moved J2 8.26 mm to (16.4, 2.19)
- moved R16 6.99 mm to (27.6, 4.60)
- moved IC1 5.43 mm to (10.3, 12.2)
- moved U$12 5.40 mm to (4.60, 15.1)
- moved C36 5.22 mm to (42.2, 1.91), turned to 180 degrees
- moved U$13 4.83 mm to (4.60, 21.3)
- moved C35 4.43 mm to (42.2, 7.94), turned to 0 degrees
- moved R18 3.84 mm to (32.5, 3.02)
- moved D3 3.52 mm to (34.4, 3.02)
- moved R17 3.37 mm to (36.4, 3.02)
- moved D4 3.21 mm to (38.3, 3.02)
- moved Y2 2.29 mm to (42.2, 4.92), turned to 90 degrees
- moved U$11 0.65 mm to (4.60, 27.5)
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Connections:
- net GATE: now also T3.G; no longer T1.G
- net GATE2: now also T1.G; no longer T2.G
- net GND: now also U1.4
- net HOT: now also T1.A2, T3.A2; no longer T1.T2, T2.T2
- net LOAD1: now also T3.A1; no longer T1.T1
- net LOAD2: now also T1.A1; no longer T2.T1
- net MISO: now also U1.2
- net MOSI: now also U1.5
- net SCK: now also U1.6
- net VCC: now also U1.8
Routing:
- net HOT: track 109.5 -> 79.8 mm, vias 5 -> 2
- net N$24: track 0.00 -> 21.6 mm
- net N$23: track 0.00 -> 16.3 mm
- net ACTLED: track 0.00 -> 14.8 mm
- net LNKLED: track 0.00 -> 13.0 mm
- net GND: track 69.2 -> 74.4 mm
- net LOAD1: track 37.4 -> 41.5 mm, vias 0 -> 2
- net GATE2: track 24.6 -> 27.8 mm, vias 0 -> 2
- net GATE: track 23.8 -> 25.8 mm, vias 0 -> 2
- net N$12: track 0.00 -> 1.95 mm
- net N$13: track 0.00 -> 1.95 mm
- net LOAD2: track 39.1 -> 39.3 mm, vias 0 -> 2

Commit message: HEEP-414 REVB design for review :)
Parts:
- added J3: (no value), SparkFun-Connectors:1X03_NO_SILK
- moved U$13 6.84 mm to (4.13, 14.4)
- moved U$12 5.58 mm to (4.13, 20.6)
- moved R19 1.56 mm to (17.5, 19.1), turned to 0 degrees
- moved U$14 1.00 mm to (9.84, 4.13)
- moved U$11 0.79 mm to (4.13, 26.8)
- moved U$16 0.79 mm to (4.13, 3.02)
- moved U$17 0.79 mm to (4.13, 8.26)
- moved D1 0.79 mm to (12.7, 18.4)
- moved R10 0.79 mm to (14.8, 21.3)
- moved R11 0.79 mm to (12.7, 21.3)
- moved R26 0.57 mm to (43.2, 42.1)
- moved U1 0.50 mm to (18.9, 6.83), turned to 90 degrees
- moved J2 0.48 mm to (16.4, 1.71)
- moved D2 0.32 mm to (14.3, 18.4)
- moved R16 0.22 mm to (27.8, 4.76)
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Connections:
- net GND: now also U$11.GND, U$12.GND, U$13.GND, U$14.GND, U$16.GND, U$17.GND; no longer U$11.P$2, U$12.P$2, U$13.P$2, U$14.P$1, U$16.P$1, U$17.P$1
- net RA0: now also U$17.SIG; no longer U$13.P$3
- net RA1: now also U$16.SIG
- net RA2: now also U$14.SIG
- net RA3: now also U1.1
- net RA4: now also U1.7; no longer R26.2
- net RA5: now also U1.3; no longer R27.2
- net RA6: now also R27.2
- net RA7: now also R26.2
- net RB0: now also J3.3
- net RB1: now also J3.2; no longer U$14.P$2
- net RB2: now also J3.1; no longer U$16.P$2
- net RB3: now also U$11.SIG; no longer U$17.P$2
- net RB4: now also U$12.SIG; no longer U$11.P$3
- net RB5: now also U$13.SIG; no longer U$12.P$3
- net VCC: now also U$11.VCC, U$12.VCC, U$13.VCC; no longer U$11.P$1, U$12.P$1, U$13.P$1
Routing:
- net RA7: track 0.00 -> 68.3 mm, vias 0 -> 2
- net RA6: track 0.00 -> 52.8 mm, vias 0 -> 2
- net GND: track 74.4 -> 121.9 mm, vias 6 -> 12
- net MCLR: track 0.00 -> 37.5 mm, vias 0 -> 2
- net RA4: track 44.8 -> 8.97 mm, vias 1 -> 0
- net MISO: track 0.10 -> 32.0 mm, vias 0 -> 3
- net MOSI: track 5.80 -> 35.3 mm, vias 1 -> 4
- net VCC: track 53.6 -> 81.9 mm, vias 2 -> 9
- net PGC: track 0.00 -> 26.4 mm, vias 0 -> 1
- net PGD: track 0.00 -> 24.4 mm, vias 0 -> 2
- net RA5: track 30.8 -> 13.9 mm, vias 1 -> 0
- net RA3: track 0.00 -> 15.7 mm
- net RB3: track 0.00 -> 13.4 mm
- net SCK: track 19.3 -> 29.9 mm, vias 1 -> 3
- net RB0: track 0.00 -> 8.10 mm
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Other:
- board text added: "0"
- board text added: "1"
- board text added: "14"
- board text added: "15"
- board text added: "16"
- board text added: "17"
- board text added: "18"
- board text added: "19"
- board text added: "2"
- board text added: "20"
- board text added: "21"
- board text added: "6"
- board text added: "7"
- board text added: "GND"
- board text added: "MCLR"
- board text added: "PGC"
- board text added: "PGD"
- board text added: "PGM"
- board text added: "VCC"
