File: Hardware/PIC18f26k40_TPBackpack/REV B/PIC_backpack.sch (EAGLE design)
At the start: 60 parts, among them IC1 PIC18F2480-I/ML, T1 BT138-V, T2 BT138-V, U4 W5500, Y2 CRYSTAL-GROUNDEDSMD-3.2X2.5

Commit message: HEEP-414 back to work
Parts:
- removed T2: BT138-V, triac:BT138-V
- added T3: BT138, triac:BT138
- added U1: 4MB Flash, SparkFun-IC-Memory:AT25SF041
- T1: value BT138-V -> BT138; device triac:BT138-V -> triac:BT138
- U$1: value TPLINK_BACKPACK -> TPLINK_BACKPACKMINIMAL_HOLES; device Heep:TPLINK_BACKPACK -> Heep:TPLINK_BACKPACKMINIMAL_HOLES
Connections:
- net GATE: now also T3.G; no longer T1.G
- net GATE2: now also T1.G; no longer T2.G
- net GND: now also U1.GND
- net HOT: now also T3.A2; no longer T2.A2
- net LOAD1: now also T3.A1; no longer T1.A1
- net LOAD2: now also T1.A1; no longer T2.A1
- net MISO: now also U1.SO(D1)
- net MOSI: now also U1.SI(D0)
- net SCK: now also U1.SCK
- net VCC: now also U1.VCC
Other:
- moved on the sheet: T1

Commit message: HEEP-414 REVB design for review :)
Parts:
- added J3: (no value), SparkFun-Connectors:CONN_031X03_NO_SILK
Connections:
- net GND: now also U$11.GND, U$12.GND, U$13.GND, U$14.GND, U$16.GND, U$17.GND; no longer U$11.P$2, U$12.P$2, U$13.P$2, U$14.P$1, U$16.P$1, U$17.P$1
- net RA0: now also U$17.SIG; no longer U$13.P$3
- net RA1: now also U$16.SIG
- net RA2: now also U$14.SIG
- net RA3: now also U1.!CS
- net RA4: now also U1.!HOLD(D3); no longer R26.2
- net RA5: now also U1.!WP(D2); no longer R27.2
- net RA6: now also R27.2
- net RA7: now also R26.2
- net RB0: now also J3.3
- net RB1: now also J3.2; no longer U$14.P$2
- net RB2: now also J3.1; no longer U$16.P$2
- net RB3: now also U$11.SIGNAL; no longer U$17.P$2
- net RB4: now also U$12.SIGNAL; no longer U$11.P$3
- net RB5: now also U$13.SIGNAL; no longer U$12.P$3
- net VCC: now also U$11.VCC, U$12.VCC, U$13.VCC; no longer U$11.P$1, U$12.P$1, U$13.P$1
