File: Hardware/PoE_MotorDriver/Rev-B/PoE_Motor-revB.brd (EAGLE design)
At the start: 91.8 x 45.4 mm, 88 parts, among them IC2 ATMEGA32U4-MU, J6 10103594-0001LF, SW1 SPST_TACT-KMR2, T1 DMG3415U, U2 SPX3819-3.3, U3 LMV358IDGKR, U4 W5500, U8 DRV8871, U9 DRV8871, X2 J1011FHANRUN, X3 DCMOTOR, X4 DCMOTOR, Y4 8MHz

Commit message: HEEP-614 finished rev b motor driver
Parts:
- moved J5 193.6 mm to (72.7, 13.3)
- moved J4 191.2 mm to (72.7, 29.8)
- moved J3 165.2 mm to (72.7, 20.6)
- moved J2 162.9 mm to (72.7, 37.1)
- moved D3 3.82 mm to (72.7, 18.4), turned to 270 degrees
- moved D4 3.82 mm to (72.7, 11.1), turned to 270 degrees
- moved D1 1.93 mm to (72.7, 34.9), turned to 270 degrees
- moved D2 1.93 mm to (72.7, 27.6), turned to 270 degrees
- moved R31 1.93 mm to (68.9, 30.8)
- moved R32 1.91 mm to (68.9, 15.2)
- moved R11 1.85 mm to (72.7, 9.53)
- moved R10 1.85 mm to (72.7, 16.8)
- moved R9 1.00 mm to (72.7, 26.0)
- moved R6 1.00 mm to (72.7, 33.3)
Connections:
- removed net 10: J4.1, U8.3
- removed net 5: J2.1, U8.2
- removed net 6: J5.1, U9.3
- removed net 9: J3.1, U9.2
- net EN1: now also D1.A, J2.1, U8.2
- net EN2: now also D2.A, J4.1, U8.3
- net EN3: now also D3.A, J3.1, U9.2
- net EN4: now also D4.A, J5.1, U9.3
Routing:
- net EN1: track 11.6 -> 54.2 mm, vias 1 -> 2
- net EN2: track 11.5 -> 48.5 mm, vias 1 -> 2
- net EN3: track 11.6 -> 35.2 mm, vias 1 -> 2
- net EN4: track 11.5 -> 30.0 mm, vias 1 -> 2
- net CMP: track 14.2 -> 6.95 mm
- net N$33: track 7.29 -> 10.7 mm
- net N$34: track 8.48 -> 10.9 mm
- net 5: track 2.20 -> 0.00 mm, vias 1 -> 0
- net N$9: track 0.00 -> 1.67 mm
- net N$8: track 0.00 -> 1.67 mm
- net N$7: track 0.00 -> 1.67 mm
- net N$5: track 0.00 -> 1.67 mm
- net 10: track 1.57 -> 0.00 mm, vias 1 -> 0
- net 9: track 0.94 -> 0.00 mm, vias 1 -> 0
- net 6: track 0.94 -> 0.00 mm, vias 1 -> 0
Other:
- board text added: "MotorDriver Rev-B"
- board text removed: "+ -"
- board text removed: "MotorDriver Rev-C"

Commit message: HEEP-651 updated capacitor voltage ratings to reflect true minimum requirements
Parts:
- C4: value 10µF 50V -> 10µF 25V
- C53, C55: value 0.1uF/50V -> 0.1uF/25V
Changed lines of the file:
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@@
 </element>
 <element name="U$19" library="Heep" package="QFN-16" value="BUCK_CONVERTER" x="53.0225" y="16.1925"/>
-<element name="C4" library="microbuilder" package="0603-MINI" value="10µF 50V" x="48.5775" y="18.0975" rot="R180"/>
+<element name="C4" library="microbuilder" package="0603-MINI" value="10µF 25V" x="48.5775" y="18.0975" rot="R180"/>
 <element name="C12" library="microbuilder" package="0603-MINI" value="22uF 10V" x="46.99" y="21.9075" rot="R270"/>
 <element name="C13" library="microbuilder" package="0603-MINI" value="22uF 10V" x="48.895" y="21.9075" rot="R270"/>
@@
 </element>
 <element name="U8" library="microbuilder" package="HSOP8" value="DRV8871" x="80.01" y="34.925" rot="R270"/>
-<element name="C53" library="microbuilder" package="0603-NO" value="0.1uF/50V" x="80.225" y="30.48" rot="R180"/>
+<element name="C53" library="microbuilder" package="0603-NO" value="0.1uF/25V" x="80.225" y="30.48" rot="R180"/>
 <element name="C54" library="microbuilder" package="PANASONIC_D" value="22uF/63V" x="80.01" y="25.4"/>
 <element name="R31" library="adafruit" package="0805-THM" value="30K" x="68.8975" y="30.7975" rot="R90"/>
 <element name="X3" library="microbuilder" package="TERMBLOCK_1X2-3.5MM" value="DCMOTOR" x="88.5825" y="30.48" rot="R90"/>
 <element name="U9" library="microbuilder" package="HSOP8" value="DRV8871" x="79.375" y="17.78" rot="R270"/>
-<element name="C55" library="microbuilder" package="0603-NO" value="0.1uF/50V" x="79.375" y="13.335" rot="R180"/>
+<element name="C55" library="microbuilder" package="0603-NO" value="0.1uF/25V" x="79.375" y="13.335" rot="R180"/>
 <element name="C56" library="microbuilder" package="PANASONIC_D" value="22uF/63V" x="80.01" y="8.255"/>
 <element name="R32" library="adafruit" package="0805-THM" value="30K" x="68.8975" y="15.24" rot="R90"/>
