File: Hardware/PoE_RFID/REV-B/PoE_RFID.brd (EAGLE design)
At the start: 99.2 x 62.1 mm, 104 parts, among them IC2 ATMEGA32U4-MU, J6 10103594-0001LF, Q1 MMBT2222, SW1 SPST_TACT-KMR2, U1 PN532, U2 SPX3819-3.3, U3 74AHC1G125, U4 W5500, X2 J1011FHANRUN, Y1 27.12MHz, Y4 8MHz

Commit message: HEEP-651 updated capacitor voltage ratings to reflect true minimum requirements
Parts:
- D1: value (none) -> MBR120
Changed lines of the file:
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@@
 <attribute name="VALUE" x="27.93925" y="23.97525" size="0.8128" layer="27" font="vector" ratio="10" rot="R270"/>
 </element>
-<element name="D1" library="microbuilder" package="SOD-123" value="" x="8.89" y="31.75" smashed="yes" rot="R270">
+<element name="D1" library="microbuilder" package="SOD-123" value="MBR120" x="8.89" y="31.75" smashed="yes" rot="R270">
 <attribute name="NAME" x="9.906" y="33.02" size="0.8128" layer="25" ratio="18" rot="R270"/>
 <attribute name="VALUE" x="7.112" y="33.02" size="0.4064" layer="27" ratio="10" rot="R270"/>
