File: Hardware/PLC_32u4/REV-A/PLC_32u4_REV-A.brd (EAGLE design)
At the start: 45 x 57.5 mm, 71 parts, among them IC1 ATMEGA32U4-MU, J18 10103594-0001LF, SW2 SPST_TACT-KMR2, T2 BT138, T4 BT138, U1 3.3V, U2 W5500, Y1 CRYSTAL-GROUNDEDSMD-3.2X2.5, Y2 8MHz

Commit message: HEEP-726 PLC 32u4 design
Parts:
- added U$4: JST_MINI_MICRO, Heep:3P_JST1.0
- moved D19 25.6 mm to (2.06, 0.95), turned to 90 degrees
- moved R58 23.0 mm to (2.07, 2.27), turned to 180 degrees
- moved U$3 4.53 mm to (15.7, 21.5)
- moved U$31 0.64 mm to (8.41, 3.81)
Connections:
- net 0: now also U$4.GND
- net 1: now also U$4.SIG
- net GND: now also U$4.VCC
Routing:
- net 1: track 0.00 -> 7.49 mm
- net 0: track 0.00 -> 7.11 mm
- net 13: track 18.8 -> 23.7 mm
- net SCL: track 5.36 -> 8.74 mm
- net SDA: track 5.01 -> 7.95 mm
- net GND: track 40.1 -> 42.6 mm, vias 15 -> 17
- net +3V3: track 178.7 -> 181.0 mm, vias 18 -> 20
- net D4: track 44.8 -> 45.9 mm
- net N$46: track 2.15 -> 1.40 mm
Other:
- board text added: "RX"
- board text added: "TX"
