File: Hardware/PLC_32u4/REV-A/PLC_32u4_REV-A.sch (EAGLE design)
At the start: 70 parts, among them IC1 ATMEGA32U4-MU, J18 10103594-0001LF, SW2 SPST_TACT-KMR2, T2 BT138, T4 BT138, U1 3.3V, U2 W5500, Y1 CRYSTAL-GROUNDEDSMD-3.2X2.5, Y2 8MHz

Commit message: HEEP-726 PLC 32u4 design
Parts:
- added U$4: JST_MINI_MICRO, Heep:JST_MINI_MICRO
Connections:
- net 0: now also U$4.GND
- net 1: now also U$4.SIGNAL
- net GND: now also U$4.VCC
Changed lines of the file:
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@@
 <?xml version="1.0" encoding="utf-8"?>
 <!DOCTYPE eagle SYSTEM "eagle.dtd">
-<eagle version="8.6.0">
+<eagle version="8.6.3">
 <drawing>
 <settings>
@@
 <part name="GND7" library="SparkFun-Aesthetics" deviceset="GND" device=""/>
 <part name="+3V11" library="supply1" deviceset="+3V3" device=""/>
+<part name="U$4" library="Heep" deviceset="JST_MINI_MICRO" device=""/>
+<part name="GND5" library="SparkFun-Aesthetics" deviceset="GND" device=""/>
 </parts>
 <sheets>
@@
 <instance part="GND7" gate="1" x="144.78" y="71.12" rot="R90"/>
 <instance part="+3V11" gate="G$1" x="139.7" y="78.74" rot="MR0"/>
+<instance part="U$4" gate="G$1" x="144.78" y="116.84" rot="R90"/>
+<instance part="GND5" gate="1" x="144.78" y="129.54" rot="R180"/>
 </instances>
 <busses>
@@
 <pinref part="GND7" gate="1" pin="GND"/>
 </segment>
+<segment>
+<pinref part="U$4" gate="G$1" pin="VCC"/>
+<pinref part="GND5" gate="1" pin="GND"/>
+<wire x1="144.78" y1="127" x2="144.78" y2="121.92" width="0.1524" layer="91"/>
+</segment>
 </net>
 <net name="INT" class="0">
@@
 <label x="38.1" y="269.24" size="1.778" layer="95"/>
 </segment>
+<segment>
+<wire x1="144.78" y1="116.84" x2="160.02" y2="116.84" width="0.1524" layer="91"/>
+<pinref part="U$4" gate="G$1" pin="SIGNAL"/>
+</segment>
 </net>
 <net name="0" class="0">
@@
 <label x="38.1" y="266.7" size="1.778" layer="95"/>
 </segment>
-</net>
+<segment>
+<wire x1="160.02" y1="119.38" x2="144.78" y2="119.38" width="0.1524" layer="91"/>
+<pinref part="U$4" gate="G$1" pin="GND"/>
+</segment>
+</net>
