File: Hardware/NodeMCU Bases/2 Button Base/2ButtonBase.brd (EAGLE design)
At the start: 48.3 x 25.4 mm, 4 parts

Commit message: HEEP-908 2 button for allpcb
Routing:
- net N$1: track 12.4 -> 11.7 mm
- added copper zone on layer 16, net GND
Other:
- board text added: "USB"
Changed lines of the file:
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@@
 <text x="8" y="7.2" size="2.54" layer="21">A</text>
 <text x="33.7" y="7.2" size="2.54" layer="21">B</text>
+<text x="-1.5875" y="6.985" size="1.27" layer="21">USB</text>
+<wire x1="0" y1="9.525" x2="-1.905" y2="9.525" width="0.1524" layer="21"/>
+<wire x1="-1.27" y1="8.89" x2="-1.905" y2="9.525" width="0.1524" layer="21"/>
+<wire x1="-1.905" y1="9.525" x2="-1.27" y2="10.16" width="0.1524" layer="21"/>
+<wire x1="0" y1="5.715" x2="-1.905" y2="5.715" width="0.1524" layer="21"/>
+<wire x1="-1.27" y1="5.08" x2="-1.905" y2="5.715" width="0.1524" layer="21"/>
+<wire x1="-1.905" y1="5.715" x2="-1.27" y2="6.35" width="0.1524" layer="21"/>
+<text x="-1.5875" y="24.13" size="1.27" layer="21">USB</text>
+<wire x1="0" y1="26.67" x2="-1.905" y2="26.67" width="0.1524" layer="21"/>
+<wire x1="-1.27" y1="26.035" x2="-1.905" y2="26.67" width="0.1524" layer="21"/>
+<wire x1="-1.905" y1="26.67" x2="-1.27" y2="27.305" width="0.1524" layer="21"/>
+<wire x1="0" y1="22.86" x2="-1.905" y2="22.86" width="0.1524" layer="21"/>
+<wire x1="-1.27" y1="22.225" x2="-1.905" y2="22.86" width="0.1524" layer="21"/>
+<wire x1="-1.905" y1="22.86" x2="-1.27" y2="23.495" width="0.1524" layer="21"/>
 </plain>
 <attributes>
@@
 <contactref element="U$1" pad="D5"/>
 <contactref element="S1" pad="1"/>
-<wire x1="21.415" y1="27.94" x2="21.59" y2="26.67" width="0.4064" layer="1"/>
-<wire x1="21.59" y1="26.67" x2="22.86" y2="25.4" width="0.4064" layer="1"/>
-<wire x1="22.86" y1="25.4" x2="24.13" y2="25.4" width="0.4064" layer="1"/>
-<wire x1="24.13" y1="25.4" x2="28.04" y2="21.49" width="0.4064" layer="1"/>
-<wire x1="28.04" y1="21.49" x2="28.04" y2="19.01" width="0.4064" layer="1"/>
+<wire x1="28.04" y1="21.315" x2="28.04" y2="19.01" width="0.4064" layer="16"/>
+<wire x1="21.415" y1="27.94" x2="22.089" y2="27.266" width="0.4064" layer="16"/>
+<wire x1="22.089" y1="27.266" x2="22.089" y2="27.167075" width="0.4064" layer="16"/>
+<wire x1="22.089" y1="27.167075" x2="23.182075" y2="26.074" width="0.4064" layer="16"/>
+<wire x1="23.182075" y1="26.074" x2="23.281" y2="26.074" width="0.4064" layer="16"/>
+<wire x1="23.281" y1="26.074" x2="28.04" y2="21.315" width="0.4064" layer="16"/>
 </signal>
 <signal name="N$2">
 <contactref element="U$1" pad="D6"/>
 <contactref element="S2" pad="1"/>
-<wire x1="15.14" y1="14.01" x2="17.78" y2="16.65" width="0.4064" layer="1"/>
-<wire x1="17.78" y1="16.65" x2="17.78" y2="25.4" width="0.4064" layer="1"/>
-<wire x1="17.78" y1="25.4" x2="19.05" y2="26.67" width="0.4064" layer="1"/>
-<wire x1="19.05" y1="26.67" x2="18.875" y2="27.94" width="0.4064" layer="1"/>
+<wire x1="15.14" y1="14.01" x2="17.78" y2="16.65" width="0.4064" layer="16"/>
+<wire x1="17.78" y1="26.746075" x2="18.201" y2="27.167075" width="0.4064" layer="16"/>
+<wire x1="18.201" y1="27.167075" x2="18.201" y2="27.266" width="0.4064" layer="16"/>
+<wire x1="18.201" y1="27.266" x2="18.875" y2="27.94" width="0.4064" layer="16"/>
+<wire x1="17.78" y1="16.65" x2="17.78" y2="26.746075" width="0.4064" layer="16"/>
 </signal>
 <signal name="GND">
@@
 <vertex x="-5.08" y="1.27"/>
 </polygon>
+<polygon width="0.4064" layer="16">
+<vertex x="-7.62" y="33.02"/>
+<vertex x="48.26" y="33.02"/>
+<vertex x="48.26" y="-1.27"/>
+<vertex x="-7.62" y="-1.27"/>
+</polygon>
 </signal>
