File: Hardware/PoE_MotorDriver/Rev-C/PoE_Motor-revC.brd (EAGLE design)
At the start: 66.4 x 45.4 mm, 79 parts, among them IC2 ATMEGA32U4-MU, J6 10103594-0001LF, SW1 SPST_TACT-KMR2, U1 DRV8871, U2 DRV8871, U4 W5500, X1 DCMOTOR, X2 J1011FHY931147C, X5 DCMOTOR, Y4 8MHz

Commit message: HEEP-728 made values more readable on brd file
Parts:
- 25MHZ: value CRYSTAL-GROUNDEDSMD-3.2X2.5 -> 25MHZ
- D10, D8: value (none) -> GRN
- D11, D9: value (none) -> YELLOW
- D5: value (none) -> RED
- SW1: value SPST_TACT-KMR2 -> TACTILE
Other:
- board text removed: "+"
- board text removed: "10"
- board text removed: "11"
- board text removed: "12"
- board text removed: "9"
- board text removed: "A0"
- board text removed: "A1"
- board text removed: "A2"
- board text removed: "A3"
- board text removed: "A4"
- board text removed: "A5"
