File: Hardware/PoE_Maglock/Rev-G/PoE_Mag-revG.sch (EAGLE design)
At the start: 89 parts, among them IC2 ATMEGA32U4-MU, J14 1X2-3.5MM, J15 1X2-3.5MM, J16 1X2-3.5MM, J17 1X2-3.5MM, J2 1X2-3.5MM, J3 1X2-3.5MM, J4 1X2-3.5MM, J5 1X2-3.5MM, J6 10103594-0001LF, Q1 35A/25V/8.5mΩ, Q3 35A/25V/8.5mΩ, Q5 35A/25V/8.5mΩ, Q6 35A/25V/8.5mΩ, SW1 SPST_TACT-KMR2, U4 W5500, X2 J1011FHY931147C, Y4 8MHz

Commit message: HEEP-1046 before rotating buck circuit 90 degrees
Parts:
- added J11: 1X2-3.5MM, adafruit:1X2-3.5MM
Connections:
- removed net N$2: R14.1, X2.POE+
- new net POE+: D12.C, R14.1, X2.POE+
- net GND: now also J11.2
- net VBAT: now also J11.1; no longer D12.C
Other:
- note added: "POST FUSE PWR"
Changed lines of the file:
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@@
 <part name="U$17" library="microbuilder" deviceset="GND" device=""/>
 <part name="D12" library="microbuilder" deviceset="DIODE" device="SOD-123" value="PMEG4030ER"/>
-<part name="U$16" library="microbuilder" deviceset="VBAT" device=""/>
+<part name="J11" library="adafruit" library_urn="urn:adsk.eagle:library:420" deviceset="1X2" device="-3.5MM"/>
+<part name="GND10" library="supply1" deviceset="GND" device=""/>
+<part name="U$18" library="microbuilder" deviceset="VBAT" device=""/>
 </parts>
 <sheets>
@@
 <text x="360.68" y="317.5" size="2.54" layer="97">I2C BREAKOUT</text>
 <text x="398.78" y="317.5" size="2.54" layer="97">SERIAL BREAKOUT</text>
+<text x="452.12" y="317.5" size="2.54" layer="97">POST FUSE PWR</text>
 </plain>
 <instances>
@@
 <instance part="U$17" gate="G$1" x="43.18" y="218.44"/>
 <instance part="D12" gate="G$1" x="53.34" y="226.06"/>
-<instance part="U$16" gate="G$1" x="66.04" y="226.06" rot="R270"/>
+<instance part="J11" gate="G$1" x="457.2" y="297.18"/>
+<instance part="GND10" gate="1" x="452.12" y="289.56"/>
+<instance part="U$18" gate="G$1" x="452.12" y="307.34"/>
 </instances>
 <busses>
@@
 <junction x="43.18" y="220.98"/>
 </segment>
+<segment>
+<pinref part="J11" gate="G$1" pin="2"/>
+<pinref part="GND10" gate="1" pin="GND"/>
+<wire x1="452.12" y1="292.1" x2="452.12" y2="297.18" width="0.1524" layer="91"/>
+</segment>
 </net>
 <net name="RD-" class="0">
@@
 </segment>
 <segment>
-<pinref part="D12" gate="G$1" pin="C"/>
-<wire x1="55.88" y1="226.06" x2="63.5" y2="226.06" width="0.1524" layer="91"/>
-<pinref part="U$16" gate="G$1" pin="VBAT"/>
+<pinref part="J11" gate="G$1" pin="1"/>
+<pinref part="U$18" gate="G$1" pin="VBAT"/>
+<wire x1="452.12" y1="304.8" x2="452.12" y2="299.72" width="0.1524" layer="91"/>
 </segment>
 </net>
@@
 </segment>
 </net>
-<net name="N$2" class="0">
+<net name="POE+" class="0">
 <segment>
 <pinref part="X2" gate="G$1" pin="POE+"/>
 <wire x1="58.42" y1="60.96" x2="45.72" y2="60.96" width="0.1524" layer="91"/>
 <pinref part="R14" gate="G$1" pin="1"/>
-</segment>
-</net>
+<label x="48.26" y="60.96" size="1.778" layer="95"/>
+</segment>
+<segment>
+<pinref part="D12" gate="G$1" pin="C"/>
+<wire x1="55.88" y1="226.06" x2="63.5" y2="226.06" width="0.1524" layer="91"/>
+<label x="58.42" y="226.568" size="1.778" layer="95"/>
+</segment>
+</net>

Commit message: HEEP-1046 stopping for the night to focus on JW
Parts:
- removed U$4: 2.1MMJACKTHM, adafruit:2.1MMJACKTHM
- added X4: (no value), microbuilder:DCBARRELPTH
Connections:
- net GND: now also X4.GND, X4.GNDBREAK; no longer U$4.RING, U$4.RING_SW
- net N$1: now also X4.PWR; no longer U$4.TIP
Changed lines of the file:
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@@
 <part name="+3V14" library="supply1" deviceset="+3V3" device=""/>
 <part name="+3V15" library="supply1" deviceset="+3V3" device=""/>
-<part name="U$4" library="adafruit" library_urn="urn:adsk.eagle:library:420" deviceset="2.1MMJACK" device="THM"/>
 <part name="U$17" library="microbuilder" deviceset="GND" device=""/>
 <part name="D12" library="microbuilder" deviceset="DIODE" device="SOD-123" value="PMEG4030ER"/>
@@
 <part name="GND10" library="supply1" deviceset="GND" device=""/>
 <part name="U$18" library="microbuilder" deviceset="VBAT" device=""/>
+<part name="X4" library="microbuilder" deviceset="DCBARREL" device="PTH"/>
 </parts>
 <sheets>
@@
 <instance part="+3V14" gate="G$1" x="444.5" y="241.3" rot="R180"/>
 <instance part="+3V15" gate="G$1" x="421.64" y="241.3" rot="R180"/>
-<instance part="U$4" gate="G$1" x="38.1" y="223.52"/>
 <instance part="U$17" gate="G$1" x="43.18" y="218.44"/>
 <instance part="D12" gate="G$1" x="53.34" y="226.06"/>
@@
 <instance part="GND10" gate="1" x="452.12" y="289.56"/>
 <instance part="U$18" gate="G$1" x="452.12" y="307.34"/>
+<instance part="X4" gate="G$1" x="33.02" y="223.52"/>
 </instances>
 <busses>
@@
 </segment>
 <segment>
-<pinref part="U$4" gate="G$1" pin="RING"/>
 <pinref part="U$17" gate="G$1" pin="GND"/>
-<pinref part="U$4" gate="G$1" pin="RING_SW"/>
-<wire x1="43.18" y1="223.52" x2="43.18" y2="220.98" width="0.1524" layer="91"/>
-<junction x="43.18" y="220.98"/>
+<wire x1="35.56" y1="223.52" x2="35.56" y2="220.98" width="0.1524" layer="91"/>
+<junction x="35.56" y="220.98"/>
+<pinref part="X4" gate="G$1" pin="GNDBREAK"/>
+<pinref part="X4" gate="G$1" pin="GND"/>
+<wire x1="35.56" y1="220.98" x2="43.18" y2="220.98" width="0.1524" layer="91"/>
 </segment>
 <segment>
@@
 <net name="N$1" class="0">
 <segment>
-<pinref part="U$4" gate="G$1" pin="TIP"/>
 <pinref part="D12" gate="G$1" pin="A"/>
-<wire x1="43.18" y1="226.06" x2="50.8" y2="226.06" width="0.1524" layer="91"/>
-</segment>
-</net>
+<wire x1="35.56" y1="226.06" x2="50.8" y2="226.06" width="0.1524" layer="91"/>
+<pinref part="X4" gate="G$1" pin="PWR"/>
+</segment>
+</net>

Commit message: HEEP-1046 added terminal block silks and ground cheese vias for mag
Connections:
- net GND: now also J11.1; no longer J11.2
- net VBAT: now also J11.2; no longer J11.1
Changed lines of the file:
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@@
 <grid distance="0.1" unitdist="inch" unit="inch" style="lines" multiple="1" display="no" altdistance="0.01" altunitdist="inch" altunit="inch"/>
 <layers>
-<layer number="1" name="Top" color="4" fill="1" visible="yes" active="no"/>
-<layer number="16" name="Bottom" color="1" fill="1" visible="yes" active="no"/>
-<layer number="17" name="Pads" color="2" fill="1" visible="yes" active="no"/>
-<layer number="18" name="Vias" color="2" fill="1" visible="yes" active="no"/>
-<layer number="19" name="Unrouted" color="15" fill="1" visible="yes" active="no"/>
-<layer number="20" name="Dimension" color="24" fill="1" visible="yes" active="no"/>
-<layer number="21" name="tPlace" color="14" fill="1" visible="yes" active="no"/>
-<layer number="22" name="bPlace" color="7" fill="1" visible="yes" active="no"/>
-<layer number="23" name="tOrigins" color="15" fill="1" visible="yes" active="no"/>
-<layer number="24" name="bOrigins" color="15" fill="1" visible="yes" active="no"/>
-<layer number="25" name="tNames" color="7" fill="1" visible="yes" active="no"/>
-<layer number="26" name="bNames" color="7" fill="1" visible="yes" active="no"/>
-<layer number="27" name="tValues" color="15" fill="1" visible="yes" active="no"/>
-<layer number="28" name="bValues" color="7" fill="1" visible="yes" active="no"/>
+<layer number="1" name="Top" color="4" fill="1" visible="no" active="no"/>
+<layer number="16" name="Bottom" color="1" fill="1" visible="no" active="no"/>
+<layer number="17" name="Pads" color="2" fill="1" visible="no" active="no"/>
+<layer number="18" name="Vias" color="2" fill="1" visible="no" active="no"/>
+<layer number="19" name="Unrouted" color="15" fill="1" visible="no" active="no"/>
+<layer number="20" name="Dimension" color="24" fill="1" visible="no" active="no"/>
+<layer number="21" name="tPlace" color="14" fill="1" visible="no" active="no"/>
+<layer number="22" name="bPlace" color="7" fill="1" visible="no" active="no"/>
+<layer number="23" name="tOrigins" color="15" fill="1" visible="no" active="no"/>
+<layer number="24" name="bOrigins" color="15" fill="1" visible="no" active="no"/>
+<layer number="25" name="tNames" color="7" fill="1" visible="no" active="no"/>
+<layer number="26" name="bNames" color="7" fill="1" visible="no" active="no"/>
+<layer number="27" name="tValues" color="15" fill="1" visible="no" active="no"/>
+<layer number="28" name="bValues" color="7" fill="1" visible="no" active="no"/>
 <layer number="29" name="tStop" color="7" fill="3" visible="no" active="no"/>
 <layer number="30" name="bStop" color="7" fill="6" visible="no" active="no"/>
@@
 <layer number="35" name="tGlue" color="7" fill="4" visible="no" active="no"/>
 <layer number="36" name="bGlue" color="7" fill="5" visible="no" active="no"/>
-<layer number="37" name="tTest" color="7" fill="1" visible="yes" active="no"/>
-<layer number="38" name="bTest" color="7" fill="1" visible="yes" active="no"/>
+<layer number="37" name="tTest" color="7" fill="1" visible="no" active="no"/>
+<layer number="38" name="bTest" color="7" fill="1" visible="no" active="no"/>
 <layer number="39" name="tKeepout" color="4" fill="11" visible="no" active="no"/>
 <layer number="40" name="bKeepout" color="1" fill="11" visible="no" active="no"/>
@@
 <layer number="44" name="Drills" color="7" fill="1" visible="no" active="no"/>
 <layer number="45" name="Holes" color="7" fill="1" visible="no" active="no"/>
-<layer number="46" name="Milling" color="3" fill="1" visible="yes" active="no"/>
-<layer number="47" name="Measures" color="7" fill="1" visible="yes" active="no"/>
-<layer number="48" name="Document" color="7" fill="1" visible="yes" active="no"/>
-<layer number="49" name="Reference" color="7" fill="1" visible="yes" active="no"/>
-<layer number="50" name="dxf" color="7" fill="1" visible="yes" active="no"/>
-<layer number="51" name="tDocu" color="7" fill="1" visible="yes" active="no"/>
-<layer number="52" name="bDocu" color="7" fill="1" visible="yes" active="no"/>
-<layer number="53" name="tGND_GNDA" color="7" fill="9" visible="yes" active="no"/>
-<layer number="54" name="bGND_GNDA" color="1" fill="9" visible="yes" active="no"/>
-<layer number="56" name="wert" color="7" fill="1" visible="yes" active="no"/>
-<layer number="57" name="tCAD" color="7" fill="1" visible="yes" active="no"/>
-<layer number="59" name="tCarbon" color="7" fill="1" visible="yes" active="no"/>
-<layer number="60" name="bCarbon" color="7" fill="1" visible="yes" active="no"/>
+<layer number="46" name="Milling" color="3" fill="1" visible="no" active="no"/>
+<layer number="47" name="Measures" color="7" fill="1" visible="no" active="no"/>
+<layer number="48" name="Document" color="7" fill="1" visible="no" active="no"/>
+<layer number="49" name="Reference" color="7" fill="1" visible="no" active="no"/>
+<layer number="50" name="dxf" color="7" fill="1" visible="no" active="no"/>
+<layer number="51" name="tDocu" color="7" fill="1" visible="no" active="no"/>
+<layer number="52" name="bDocu" color="7" fill="1" visible="no" active="no"/>
+<layer number="53" name="tGND_GNDA" color="7" fill="9" visible="no" active="no"/>
+<layer number="54" name="bGND_GNDA" color="1" fill="9" visible="no" active="no"/>
+<layer number="56" name="wert" color="7" fill="1" visible="no" active="no"/>
+<layer number="57" name="tCAD" color="7" fill="1" visible="no" active="no"/>
+<layer number="59" name="tCarbon" color="7" fill="1" visible="no" active="no"/>
+<layer number="60" name="bCarbon" color="7" fill="1" visible="no" active="no"/>
 <layer number="90" name="Modules" color="5" fill="1" visible="yes" active="yes"/>
 <layer number="91" name="Nets" color="2" fill="1" visible="yes" active="yes"/>
@@
 <part name="D12" library="microbuilder" deviceset="DIODE" device="SOD-123" value="PMEG4030ER"/>
 <part name="J11" library="adafruit" library_urn="urn:adsk.eagle:library:420" deviceset="1X2" device="-3.5MM"/>
+<part name="X4" library="microbuilder" deviceset="DCBARREL" device="PTH"/>
 <part name="GND10" library="supply1" deviceset="GND" device=""/>
-<part name="U$18" library="microbuilder" deviceset="VBAT" device=""/>
-<part name="X4" library="microbuilder" deviceset="DCBARREL" device="PTH"/>
+<part name="U$4" library="microbuilder" deviceset="VBAT" device=""/>
 </parts>
 <sheets>
@@
 <instance part="D12" gate="G$1" x="53.34" y="226.06"/>
 <instance part="J11" gate="G$1" x="457.2" y="297.18"/>
-<instance part="GND10" gate="1" x="452.12" y="289.56"/>
-<instance part="U$18" gate="G$1" x="452.12" y="307.34"/>
 <instance part="X4" gate="G$1" x="33.02" y="223.52"/>
+<instance part="GND10" gate="1" x="452.12" y="307.34" rot="R180"/>
+<instance part="U$4" gate="G$1" x="452.12" y="289.56" rot="R180"/>
 </instances>
 <busses>
@@
 </segment>
 <segment>
-<pinref part="J11" gate="G$1" pin="2"/>
+<pinref part="J11" gate="G$1" pin="1"/>
+<wire x1="452.12" y1="304.8" x2="452.12" y2="299.72" width="0.1524" layer="91"/>
 <pinref part="GND10" gate="1" pin="GND"/>
-<wire x1="452.12" y1="292.1" x2="452.12" y2="297.18" width="0.1524" layer="91"/>
 </segment>
 </net>
@@
 </segment>
 <segment>
-<pinref part="J11" gate="G$1" pin="1"/>
-<pinref part="U$18" gate="G$1" pin="VBAT"/>
-<wire x1="452.12" y1="304.8" x2="452.12" y2="299.72" width="0.1524" layer="91"/>
-</segment>
-</net>
+<pinref part="J11" gate="G$1" pin="2"/>
+<wire x1="452.12" y1="292.1" x2="452.12" y2="297.18" width="0.1524" layer="91"/>
+<pinref part="U$4" gate="G$1" pin="VBAT"/>
+</segment>
+</net>

Commit message: HEEP-1046 done for now. dylan to review
Parts:
- removed D12: PMEG4030ER, microbuilder:DIODESOD-123
Connections:
- removed net N$1: D12.A, X4.PWR
- net A0: now also X3.2
- net A1: now also X1.2
- net POE+: now also X4.PWR; no longer D12.C
Changed lines of the file:
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@@
 <part name="+3V15" library="supply1" deviceset="+3V3" device=""/>
 <part name="U$17" library="microbuilder" deviceset="GND" device=""/>
-<part name="D12" library="microbuilder" deviceset="DIODE" device="SOD-123" value="PMEG4030ER"/>
 <part name="J11" library="adafruit" library_urn="urn:adsk.eagle:library:420" deviceset="1X2" device="-3.5MM"/>
 <part name="X4" library="microbuilder" deviceset="DCBARREL" device="PTH"/>
@@
 <text x="83.82" y="251.46" size="2.54" layer="94" ratio="15" align="center">POWER SUPPLY: 3.3V BUCK</text>
 <text x="60.96" y="238.76" size="1.778" layer="97">VBAT is POE Voltage</text>
-<text x="370.84" y="259.08" size="2.54" layer="97">ANALOG BREAKOUTS</text>
+<text x="419.1" y="264.16" size="2.54" layer="97">ANALOG BREAKOUTS</text>
 <text x="299.72" y="190.5" size="2.54" layer="97">MOSFET OUTPUTS</text>
 <text x="360.68" y="317.5" size="2.54" layer="97">I2C BREAKOUT</text>
@@
 <instance part="+3V15" gate="G$1" x="421.64" y="241.3" rot="R180"/>
 <instance part="U$17" gate="G$1" x="43.18" y="218.44"/>
-<instance part="D12" gate="G$1" x="53.34" y="226.06"/>
 <instance part="J11" gate="G$1" x="457.2" y="297.18"/>
 <instance part="X4" gate="G$1" x="33.02" y="223.52"/>
@@
 <label x="292.1" y="327.66" size="1.778" layer="95"/>
 </segment>
-<segment>
-<wire x1="363.22" y1="248.92" x2="353.06" y2="248.92" width="0.1524" layer="91"/>
-<label x="353.06" y="248.92" size="1.778" layer="95"/>
-</segment>
 </net>
 <net name="A2" class="0">
@@
 <label x="292.1" y="325.12" size="1.778" layer="95"/>
 </segment>
-<segment>
-<wire x1="363.22" y1="246.38" x2="353.06" y2="246.38" width="0.1524" layer="91"/>
-<label x="353.06" y="246.38" size="1.778" layer="95"/>
-</segment>
 </net>
 <net name="A1" class="0">
@@
 </segment>
 <segment>
-<wire x1="363.22" y1="243.84" x2="353.06" y2="243.84" width="0.1524" layer="91"/>
-<label x="353.06" y="243.84" size="1.778" layer="95"/>
+<pinref part="X1" gate="G$1" pin="2"/>
+<wire x1="421.64" y1="246.38" x2="411.48" y2="246.38" width="0.1524" layer="91"/>
+<label x="414.02" y="246.38" size="1.778" layer="95"/>
 </segment>
 </net>
@@
 </segment>
 <segment>
-<wire x1="363.22" y1="241.3" x2="353.06" y2="241.3" width="0.1524" layer="91"/>
-<label x="353.06" y="241.3" size="1.778" layer="95"/>
+<pinref part="X3" gate="G$1" pin="2"/>
+<wire x1="444.5" y1="246.38" x2="436.88" y2="246.38" width="0.1524" layer="91"/>
+<label x="439.42" y="246.38" size="1.778" layer="95"/>
 </segment>
 </net>
@@
 </segment>
 <segment>
-<pinref part="D12" gate="G$1" pin="C"/>
-<wire x1="55.88" y1="226.06" x2="63.5" y2="226.06" width="0.1524" layer="91"/>
-<label x="58.42" y="226.568" size="1.778" layer="95"/>
-</segment>
-</net>
-<net name="N$1" class="0">
-<segment>
-<pinref part="D12" gate="G$1" pin="A"/>
+<label x="45.72" y="226.568" size="1.778" layer="95"/>
+<pinref part="X4" gate="G$1" pin="PWR"/>
 <wire x1="35.56" y1="226.06" x2="50.8" y2="226.06" width="0.1524" layer="91"/>
-<pinref part="X4" gate="G$1" pin="PWR"/>
-</segment>
-</net>
+</segment>
+</net>
